File: Hardware/SparkFun_Artemis_Global_Tracker.brd (EAGLE design)
At the start: 50.8 x 63.5 mm, 207 parts, among them J1 IRIDIUM_9603N, J2 USB-C, J6 U.FL, J7 ANTENNA-GROUNDEDEDGE_SMA, J8 STANDOFFS_M2X0.4_STEEL_6MM, J9 STANDOFFS_M2X0.4_STEEL_6MM, Q1 5.8A/30V/35mΩ, Q2 20V/4.2A/52mΩ/1.4W, Q3 20V/4.2A/52mΩ/1.4W, Q4 600mA/40V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

Commit message: silk updates almost done
Parts:
- removed U$29: (no value), Solar_0.03:SOLAR0
- removed U$59: (no value), GND:GND0
- removed U$60: (no value), VIN:VIN0
- added 3V3SW, D17, D41: (no value), SparkFun-Connectors:PAD.03X.05
- added U$28: (no value), output:#VIN#3#0
- added U$40: (no value), output:#5#3V#0
- added U$41: (no value), output:#D41#0
- added U$42: (no value), output:#RX0#0
- added U$54: (no value), output:#_EN_#0
- added U$55: (no value), output:#SOLAR#0
- added U$66: (no value), output:#6V_MAX#0
- added U$75: (no value), output:#COPI#5
- added U$76, U$77, U$78: (no value), output:#GND#152
- added U$8: (no value), output:#3V3SW#0
- U$1: device 60mA:60MA0 -> output:SUPERCAPACITOR151
- U$12: device Labels-0_04:GND1 -> output:#D4#0
- U$13: device 150mA:150MA0 -> output:SUPERCAPACITOR151
- U$14: device Charge:CHARGE0 -> output:10F_2#7V152
- U$15: device Current:CURRENT0 -> output:10F_2#7V152
- U$16: device TX0:TX00 -> output:#LIPO#163
- U$17: device Labels-0_04:GND1 -> output:#3V3#153
- U$20: device Labels-0_04:3#3V2 -> output:#GND#0
- U$21: device Labels-0_04:3#3V2 -> output:#SDA#153
- U$22: device Labels-0_04:GND1 -> output:#SCL#154
- U$23: device RX0:RX00 -> output:#TX0#163
- U$26: device Labels-0_04:SCL9 -> output:#_RST##156
- U$27: device Labels-0_04:SDA8 -> output:#EN#157
- U$3: device Labels-0_04:GND1 -> output:#3V3#0
- U$31: device SCK_BOT:SCK0 -> output:SUPERCAPS6
- U$32: device 5.3V:5#3V0 -> output:#D17#0
- U$33: device Rx:RX0 -> output:#SAFEBOOT#0
- U$34: device RX0:RX00 -> output:#TX0#0
- U$35: device RX1:RX10 -> output:#TX1#0
- U$36: device SAFEBOOT:SAFEBOOT0 -> output:#GND#0
- U$37: device Tx:TX0 -> output:#RX#0
- U$38: device TX0:TX00 -> output:#RX1#0
- U$39: device TX1:TX10 -> output:#TX#0
- U$4: device Labels-0_04:3#3V2 -> output:#SDA#0
- U$43: device PWR_LED:PWR_LED0 -> output:#3V3#0
- U$44: device VBUS:VBUS0 -> output:#RESET#162
- U$45: device LiPo_0.03:LIPO0 -> output:#SOLAR#165
- U$46: device LiPo_0.03:LIPO0 -> output:#LIPO#164
- U$47: device 3.3V EN:3#3V_EN0 -> output:#MEAS#0
- U$48: device MEAS:MEAS0 -> output:#3V3_#0
- U$49: device RESET_0.03:RESET0 -> output:#RX0#163
- U$5: device SCL_BOT:SCL0 -> output:#USB#C#0
- U$53: device USB-C:USB#C0 -> output:#LIPO#0
- U$56: device USB-C_0.03:USB#C0 -> output:#USB#C#161
- U$57: device LiPo:LIPO0 -> output:#3_X_AA#0
- U$58: device RST:#RST0 -> output:#VBUS#159
- U$6: device SDA_BOT:SDA0 -> output:#SCL#0
- U$61: device 3xAA:3_X_AA0 -> output:#PWR_LED#0
- U$62: device 3xAAA:3_X_AAA0 -> output:#D35#0
- U$63: device 6VMax:6V_MAX0 -> output:#SCL#1
- U$64: device Solar:SOLAR0 -> output:#CIPO#2
- U$65: device VINdiv3:VIN#30 -> output:#3_X_AAA#0
- U$67: device D35:D350 -> output:CHARGE8
- U$69: device MISO:MISO0 -> output:CURRENT9
- U$7: device EN:EN0 -> output:#VIN#158
- U$72: device MOSI_m:MOSI0 -> output:#150MA#10
- U$74: device D4_m:D40 -> output:#60MA#151
- moved U$17 46.3 mm to (3.96, 43.2), turned to 0 degrees
- moved U$36 44.4 mm to (3.99, 45.8)
- moved U$74 42.2 mm to (13.8, 56.4), turned to 90 degrees
- moved U$67 41.6 mm to (10.7, 52.2), turned to 90 degrees
- moved U$69 41.1 mm to (9.47, 52.1), turned to 90 degrees
- moved U$31 39.4 mm to (12.2, 52.6), turned to 90 degrees
- moved U$63 38.3 mm to (47.0, 38.0)
- moved U$5 37.0 mm to (10.7, 1.40)
- moved U$64 35.4 mm to (46.6, 40.6)
- moved U$72 35.4 mm to (13.8, 47.9), turned to 90 degrees
- moved U$62 34.0 mm to (47.0, 35.5)
- moved U$38 33.2 mm to (18.1, 45.7)
- moved U$65 31.8 mm to (32.4, 3.30), turned to 0 degrees
- moved U$14 25.6 mm to (29.4, 35.9)
- moved U$27 25.5 mm to (3.43, 15.2)
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Connections:
- net 3V3SW: now also 3V3SW.1
- net ARTEMIS_D17: now also D17.1
- net ARTEMIS_D41: now also D41.1
Routing:
- net ARTEMIS_D41: track 28.5 -> 31.4 mm
- net ARTEMIS_D17: track 35.2 -> 37.4 mm
- net 3V3SW: track 49.4 -> 51.3 mm
- net N$4: track 3.59 -> 5.05 mm
- net VIN: track 76.6 -> 78.0 mm
- net GND: track 268.1 -> 267.2 mm
- net ARTEMIS_!RESET: track 95.7 -> 96.4 mm
- net N$1: track 33.0 -> 33.7 mm
- net N$11: track 5.42 -> 5.96 mm
- net 3.3V: track 202.5 -> 203.0 mm
Other:
- board text removed: "Supercapacitor 10F 2.7V"
