File: Hardware/Production/SparkFun_Artemis_Global_Tracker-Panel_v10b.brd (EAGLE design)
At the start: 115.8 x 196.9 mm, 958 parts, among them J1 IRIDIUM_9603N, J12 IRIDIUM_9603N, J16 USB-C, J17 ANTENNA-GROUNDEDEDGE_SMA, J19 U.FL, J2 USB-C, J20 STAND-OFF-REFLOW-M2.0_6.0MM_T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, J21 STAND-OFF-REFLOW-M2.0_6.0MM_T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, J25 IRIDIUM_9603N, J28 USB-C, J29 ANTENNA-GROUNDEDEDGE_SMA, J31 U.FL, J32 STAND-OFF-REFLOW-M2.0_6.0MM_T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, J33 STAND-OFF-REFLOW-M2.0_6.0MM_T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, J37 IRIDIUM_9603N, J40 USB-C, J41 ANTENNA-GROUNDEDEDGE_SMA, J43 U.FL, J44 STAND-OFF-REFLOW-M2.0_6.0MM_T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, J45 STAND-OFF-REFLOW-M2.0_6.0MM_T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, J6 U.FL, J7 ANTENNA-GROUNDEDEDGE_SMA, J8 STAND-OFF-REFLOW-M2.0_6.0MM_T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, J9 STAND-OFF-REFLOW-M2.0_6.0MM_T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, Q1 5.8A/30V/35mΩ, Q10 20V/4.2A/52mΩ/1.4W, Q11 5.8A/30V/35mΩ, Q12 20V/4.2A/52mΩ/1.4W, Q13 20V/4.2A/52mΩ/1.4W, Q14 600mA/40V, Q15 20V/4.2A/52mΩ/1.4W, Q16 5.8A/30V/35mΩ, Q17 20V/4.2A/52mΩ/1.4W, Q18 20V/4.2A/52mΩ/1.4W, Q19 600mA/40V, Q2 20V/4.2A/52mΩ/1.4W, Q20 20V/4.2A/52mΩ/1.4W, Q3 20V/4.2A/52mΩ/1.4W, Q4 600mA/40V, Q5 5.8A/30V/35mΩ, Q6 20V/4.2A/52mΩ/1.4W, Q7 20V/4.2A/52mΩ/1.4W, Q8 20V/4.2A/52mΩ/1.4W, Q9 600mA/40V, U1 CH340E_MSOP10, U10 3.3V, U11 74LVC1G04SE, U12 74LVC1G08SE, U13 LTC3225EDDB, U14 ADM4210_1TSOT6, U15 U-BLOX_ZOE_M8Q-0-10, U16 AS179-92LF, U17 MS8607-02BA01, U18 ARTEMIS_MODULESMD, U19 MCP73831, U2 LTC3225EDDB, U20 CH340E_MSOP10, U21 3.3V, U22 V_SUPERVISOR_BD48K24G_2.4V, U23 74LVC1G08SE, U24 74LVC1G04SE, U25 LTC3225EDDB, U26 ADM4210_1TSOT6, U27 U-BLOX_ZOE_M8Q-0-10, U28 AS179-92LF, U29 MS8607-02BA01, U3 ADM4210_1TSOT6, U30 ARTEMIS_MODULESMD, U31 MCP73831, U32 CH340E_MSOP10, U33 3.3V, U34 V_SUPERVISOR_BD48K24G_2.4V, U35 74LVC1G08SE, U36 74LVC1G04SE, U37 LTC3225EDDB, U38 ADM4210_1TSOT6, U39 U-BLOX_ZOE_M8Q-0-10, U4 U-BLOX_ZOE_M8Q-0-10, U40 AS179-92LF, U41 MS8607-02BA01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

Commit message: Updated current sense resistors on production panel to 0.015Ohms (RES-16305)
updated values and prod_ids on all four boards in the panel
Parts:
- R34, R64, R9, R94: value 0.012ohm -> 0.015ohm
Changed lines of the file:
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@@
 <layer number="25" name="tNames" color="7" fill="1" visible="no" active="yes"/>
 <layer number="26" name="bNames" color="7" fill="1" visible="no" active="yes"/>
-<layer number="27" name="tValues" color="7" fill="1" visible="no" active="yes"/>
+<layer number="27" name="tValues" color="7" fill="1" visible="yes" active="yes"/>
 <layer number="28" name="bValues" color="7" fill="1" visible="no" active="yes"/>
 <layer number="29" name="tStop" color="7" fill="3" visible="no" active="yes"/>
@@
 <attribute name="PROD_ID" value="RES-14962" x="35.2298" y="46.9392" size="1.778" layer="27" rot="R270" display="off"/>
 </element>
-<element name="R9" library="SparkFun-Resistors" package="0603" value="0.012ohm" x="33.0962" y="50.1904" smashed="yes" rot="R90">
+<element name="R9" library="SparkFun-Resistors" package="0603" value="0.015ohm" x="33.0962" y="50.1904" smashed="yes" rot="R90">
 <attribute name="NAME" x="34.7472" y="49.5554" size="0.8128" layer="25" font="vector" ratio="18" rot="R90"/>
-<attribute name="PROD_ID" value="RES-14691" x="33.0962" y="50.1904" size="1.778" layer="27" rot="R90" display="off"/>
+<attribute name="PROD_ID" value="RES-16305" x="33.0962" y="50.1904" size="1.778" layer="27" rot="R90" display="off"/>
 <attribute name="VALUE" value="0.012ohm" x="33.8582" y="51.9684" size="0.4064" layer="27" font="vector" ratio="10" rot="R90"/>
 </element>
@@
 <attribute name="PROD_ID" value="RES-14962" x="86.5378" y="46.9392" size="1.778" layer="27" rot="R270" display="off"/>
 </element>
-<element name="R34" library="SparkFun-Resistors" package="0603" value="0.012ohm" x="84.4042" y="50.1904" smashed="yes" rot="R90">
+<element name="R34" library="SparkFun-Resistors" package="0603" value="0.015ohm" x="84.4042" y="50.1904" smashed="yes" rot="R90">
 <attribute name="NAME" x="86.0552" y="49.5554" size="0.8128" layer="25" font="vector" ratio="18" rot="R90"/>
-<attribute name="PROD_ID" value="RES-14691" x="84.4042" y="50.1904" size="1.778" layer="27" rot="R90" display="off"/>
+<attribute name="PROD_ID" value="RES-16305" x="84.4042" y="50.1904" size="1.778" layer="27" rot="R90" display="off"/>
 <attribute name="VALUE" value="0.012ohm" x="85.1662" y="51.9684" size="0.4064" layer="27" font="vector" ratio="10" rot="R90"/>
 </element>
@@
 <attribute name="PROD_ID" value="RES-14962" x="35.2298" y="123.1392" size="1.778" layer="27" rot="R270" display="off"/>
 </element>
-<element name="R64" library="SparkFun-Resistors" package="0603" value="0.012ohm" x="33.0962" y="126.3904" smashed="yes" rot="R90">
+<element name="R64" library="SparkFun-Resistors" package="0603" value="0.015ohm" x="33.0962" y="126.3904" smashed="yes" rot="R90">
 <attribute name="NAME" x="34.7472" y="125.7554" size="0.8128" layer="25" font="vector" ratio="18" rot="R90"/>
-<attribute name="PROD_ID" value="RES-14691" x="33.0962" y="126.3904" size="1.778" layer="27" rot="R90" display="off"/>
+<attribute name="PROD_ID" value="RES-16305" x="33.0962" y="126.3904" size="1.778" layer="27" rot="R90" display="off"/>
 <attribute name="VALUE" value="0.012ohm" x="33.8582" y="128.1684" size="0.4064" layer="27" font="vector" ratio="10" rot="R90"/>
 </element>
@@
 <attribute name="PROD_ID" value="RES-14962" x="86.5378" y="123.1392" size="1.778" layer="27" rot="R270" display="off"/>
 </element>
-<element name="R94" library="SparkFun-Resistors" package="0603" value="0.012ohm" x="84.4042" y="126.3904" smashed="yes" rot="R90">
+<element name="R94" library="SparkFun-Resistors" package="0603" value="0.015ohm" x="84.4042" y="126.3904" smashed="yes" rot="R90">
 <attribute name="NAME" x="86.0552" y="125.7554" size="0.8128" layer="25" font="vector" ratio="18" rot="R90"/>
-<attribute name="PROD_ID" value="RES-14691" x="84.4042" y="126.3904" size="1.778" layer="27" rot="R90" display="off"/>
+<attribute name="PROD_ID" value="RES-16305" x="84.4042" y="126.3904" size="1.778" layer="27" rot="R90" display="off"/>
 <attribute name="VALUE" value="0.012ohm" x="85.1662" y="128.1684" size="0.4064" layer="27" font="vector" ratio="10" rot="R90"/>
 </element>

Commit message: AND Gate (U12) PROD_ID update to correct package on PANEL FILE
Note, updated both PROD ID and part value on each part of the panel.
Parts:
- U12, U23, U35, U47: value 74LVC1G08SE -> 74LVC1G08W5-7
Changed lines of the file:
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@@
 <attribute name="PROD_ID" value="HW-14879" x="37.9032" y="20.32" size="1.778" layer="27" display="off"/>
 </element>
-<element name="U12" library="SparkFun-IC-Logic" package="SOT23-5" value="74LVC1G08SE" x="36.8808" y="42.2148" smashed="yes">
+<element name="U12" library="SparkFun-IC-Logic" package="SOT23-5" value="74LVC1G08W5-7" x="36.8808" y="42.2148" smashed="yes">
 <attribute name="NAME" x="34.9758" y="42.2148" size="0.6096" layer="25" font="vector" ratio="20" rot="R90" align="bottom-center"/>
-<attribute name="PROD_ID" value="IC-10841" x="36.8808" y="42.2148" size="1.778" layer="27" font="vector" ratio="15" display="off"/>
+<attribute name="PROD_ID" value="IC-16359" x="36.8808" y="42.2148" size="1.778" layer="27" font="vector" ratio="15" display="off"/>
 <attribute name="VALUE" x="39.4208" y="42.2148" size="0.6096" layer="27" font="vector" ratio="20" rot="R90" align="bottom-center"/>
 </element>
@@
 <attribute name="PROD_ID" value="HW-14879" x="89.2112" y="20.32" size="1.778" layer="27" display="off"/>
 </element>
-<element name="U23" library="SparkFun-IC-Logic" package="SOT23-5" value="74LVC1G08SE" x="88.1888" y="42.2148" smashed="yes">
+<element name="U23" library="SparkFun-IC-Logic" package="SOT23-5" value="74LVC1G08W5-7" x="88.1888" y="42.2148" smashed="yes">
 <attribute name="NAME" x="86.2838" y="42.2148" size="0.6096" layer="25" font="vector" ratio="20" rot="R90" align="bottom-center"/>
-<attribute name="PROD_ID" value="IC-10841" x="88.1888" y="42.2148" size="1.778" layer="27" font="vector" ratio="15" display="off"/>
+<attribute name="PROD_ID" value="IC-16359" x="88.1888" y="42.2148" size="1.778" layer="27" font="vector" ratio="15" display="off"/>
 <attribute name="VALUE" x="90.7288" y="42.2148" size="0.6096" layer="27" font="vector" ratio="20" rot="R90" align="bottom-center"/>
 </element>
@@
 <attribute name="PROD_ID" value="HW-14879" x="37.9032" y="96.52" size="1.778" layer="27" display="off"/>
 </element>
-<element name="U35" library="SparkFun-IC-Logic" package="SOT23-5" value="74LVC1G08SE" x="36.8808" y="118.4148" smashed="yes">
+<element name="U35" library="SparkFun-IC-Logic" package="SOT23-5" value="74LVC1G08W5-7" x="36.8808" y="118.4148" smashed="yes">
 <attribute name="NAME" x="34.9758" y="118.4148" size="0.6096" layer="25" font="vector" ratio="20" rot="R90" align="bottom-center"/>
-<attribute name="PROD_ID" value="IC-10841" x="36.8808" y="118.4148" size="1.778" layer="27" font="vector" ratio="15" display="off"/>
+<attribute name="PROD_ID" value="IC-16359" x="36.8808" y="118.4148" size="1.778" layer="27" font="vector" ratio="15" display="off"/>
 <attribute name="VALUE" x="39.4208" y="118.4148" size="0.6096" layer="27" font="vector" ratio="20" rot="R90" align="bottom-center"/>
 </element>
@@
 <attribute name="PROD_ID" value="HW-14879" x="89.2112" y="96.52" size="1.778" layer="27" display="off"/>
 </element>
-<element name="U47" library="SparkFun-IC-Logic" package="SOT23-5" value="74LVC1G08SE" x="88.1888" y="118.4148" smashed="yes">
+<element name="U47" library="SparkFun-IC-Logic" package="SOT23-5" value="74LVC1G08W5-7" x="88.1888" y="118.4148" smashed="yes">
 <attribute name="NAME" x="86.2838" y="118.4148" size="0.6096" layer="25" font="vector" ratio="20" rot="R90" align="bottom-center"/>
-<attribute name="PROD_ID" value="IC-10841" x="88.1888" y="118.4148" size="1.778" layer="27" font="vector" ratio="15" display="off"/>
+<attribute name="PROD_ID" value="IC-16359" x="88.1888" y="118.4148" size="1.778" layer="27" font="vector" ratio="15" display="off"/>
 <attribute name="VALUE" x="90.7288" y="118.4148" size="0.6096" layer="27" font="vector" ratio="20" rot="R90" align="bottom-center"/>
 </element>
